Commit message: Add laser scan transform
- Add node to transform laser scan data from Gazebo BODY_FLU to aerospace BODY_FRD
- Add front and rear bumpers to rover model
- Update mavros launch files to use rotated laser scan data

Signed-off-by: Rhys Mainwaring <rhys.mainwaring@me.com>

File: models/rover.urdf.xacro (robot description, xacro)
@@ -41,4 +41,32 @@
       <geometry>
         <box size="${base_x_size} ${base_y_size} ${base_z_size}"/>
+      </geometry>
+    </collision>
+    <!-- front bumper -->
+    <visual>
+      <origin xyz="${(base_x_size/2 + wheel_radius)} 0 0" rpy="0 0 0" />
+      <geometry>
+        <box size="0.05 ${base_y_size} ${base_z_size/2}"/>
+      </geometry>
+      <material name="blue"/>
+    </visual>
+    <collision>
+      <origin xyz="${(base_x_size/2 + wheel_radius)} 0 0" rpy="0 0 0" />
+      <geometry>
+        <box size="0.05 ${base_y_size} ${base_z_size/2}"/>
+      </geometry>
+    </collision>
+    <!-- rear bumper -->
+    <visual>
+      <origin xyz="${-1 * (base_x_size/2 + wheel_radius)} 0 0" rpy="0 0 0" />
+      <geometry>
+        <box size="0.05 ${base_y_size} ${base_z_size/2}"/>
+      </geometry>
+      <material name="blue"/>
+    </visual>
+    <collision>
+      <origin xyz="${-1 * (base_x_size/2 + wheel_radius)} 0 0" rpy="0 0 0" />
+      <geometry>
+        <box size="0.05 ${base_y_size} ${base_z_size/2}"/>
       </geometry>
     </collision>

Commit message: Add mavros integration (#4)
* Initial support for mavros(2)

- Remove custom static broadcaster and use tf2_ros static_transform_puiblisher instead
- Correct orientation of rover and playpen model to use ENU

Signed-off-by: Rhys Mainwaring <rhys.mainwaring@me.com>

* Add mavros(2) integration

- Add launch file for a mavros node
- Add launch config yaml files and update setup.py to install
- Update README

Signed-off-by: Rhys Mainwaring <rhys.mainwaring@me.com>

* Update comments in configuration and launch files

Signed-off-by: Rhys Mainwaring <rhys.mainwaring@me.com>

* Add laser scan transform

- Add node to transform laser scan data from Gazebo BODY_FLU to aerospace BODY_FRD
- Add front and rear bumpers to rover model
- Update mavros launch files to use rotated laser scan data

Signed-off-by: Rhys Mainwaring <rhys.mainwaring@me.com>

File: models/rover.urdf.xacro (robot description, xacro)
@@ -41,4 +41,32 @@
       <geometry>
         <box size="${base_x_size} ${base_y_size} ${base_z_size}"/>
+      </geometry>
+    </collision>
+    <!-- front bumper -->
+    <visual>
+      <origin xyz="${(base_x_size/2 + wheel_radius)} 0 0" rpy="0 0 0" />
+      <geometry>
+        <box size="0.05 ${base_y_size} ${base_z_size/2}"/>
+      </geometry>
+      <material name="blue"/>
+    </visual>
+    <collision>
+      <origin xyz="${(base_x_size/2 + wheel_radius)} 0 0" rpy="0 0 0" />
+      <geometry>
+        <box size="0.05 ${base_y_size} ${base_z_size/2}"/>
+      </geometry>
+    </collision>
+    <!-- rear bumper -->
+    <visual>
+      <origin xyz="${-1 * (base_x_size/2 + wheel_radius)} 0 0" rpy="0 0 0" />
+      <geometry>
+        <box size="0.05 ${base_y_size} ${base_z_size/2}"/>
+      </geometry>
+      <material name="blue"/>
+    </visual>
+    <collision>
+      <origin xyz="${-1 * (base_x_size/2 + wheel_radius)} 0 0" rpy="0 0 0" />
+      <geometry>
+        <box size="0.05 ${base_y_size} ${base_z_size/2}"/>
       </geometry>
     </collision>
@@ -384,5 +412,5 @@
       <lock_step>1</lock_step>
       <modelXYZToAirplaneXForwardZDown>0 0 0 ${PI} 0 0</modelXYZToAirplaneXForwardZDown>
-      <gazeboXYZToNED>0 0 0 ${PI} 0 0</gazeboXYZToNED>
+      <gazeboXYZToNED>0 0 0 ${PI} 0 ${PI/2}</gazeboXYZToNED>
       <imuName>imu_sensor</imuName>
       <!--
